File: pcb/tartan.kicad_pcb (KiCad board)
At the start: 2 copper layers, 285 x 117 mm, 175 parts, among them J1 AVR_ISP_6, J2 USB_OTG, SW1 SW_Push, SW10 SW_Push, SW11 SW_Push, SW12 SW_Push, SW13 SW_Push, SW14 SW_Push, SW15 SW_Push, SW16 SW_Push, SW17 SW_Push, SW18 SW_Push, SW19 SW_Push, SW2 SW_Push, SW20 SW_Push, SW21 SW_Push, SW22 SW_Push, SW23 SW_Push, SW24 SW_Push, SW25 SW_Push, SW26 SW_Push, SW27 SW_Push, SW28 SW_Push, SW29 SW_Push, SW3 SW_Push, SW30 SW_Push, SW31 SW_Push, SW32 SW_Push, SW33 SW_Push, SW34 SW_Push, SW35 SW_Push, SW36 SW_Push, SW37 SW_Push, SW38 SW_Push, SW39 SW_Push, SW4 SW_Push, SW40 SW_Push, SW41 SW_Push, SW42 SW_Push, SW43 SW_Push, SW44 SW_Push, SW45 SW_Push, SW46 SW_Push, SW47 SW_Push, SW48 SW_Push, SW49 SW_Push, SW5 SW_Push, SW50 SW_Push, SW51 SW_Push, SW52 SW_Push, SW53 SW_Push, SW54 SW_Push, SW55 SW_Push, SW56 SW_Push, SW57 SW_Push, SW58 SW_Push, SW59 SW_Push, SW6 SW_Push, SW60 SW_Push, SW61 SW_Push, SW62 SW_Push, SW63 SW_Push, SW64 SW_Push, SW65 SW_Push, SW66 SW_Push, SW67 SW_Push, SW68 SW_Push, SW69 SW_Push, SW7 SW_Push, SW70 RESET, SW71 BOOT, SW8 SW_Push, SW9 SW_Push, U1 ATMEGA328-PU, Y1 16MHz

Commit message: fix alpha issues
Parts:
- removed the G*** at (219.0, 137.5)
- removed the G*** at (187.5, 137.3)
- removed LED1: LED, LEDs:LED_D3.0mm
- removed R5: 1.5k, Resistors_THT:R_Axial_DIN0204_L3.6mm_D1.6mm_P5.08mm_Horizontal
- SW16, SW29, SW66: footprint SMKJP:SW_Cherry_MX1A_1.00u_PCB -> SMKJP:SW_Cherry_MX1A_1.50u_PCB
- SW30, SW56: footprint SMKJP:SW_Cherry_MX1A_1.00u_PCB -> SMKJP:SW_Cherry_MX1A_1.75u_PCB
- SW57, SW58, SW59, SW61, SW62, SW63, SW64: footprint SMKJP:SW_Cherry_MX1A_1.00u_PCB -> SMKJP:SW_Cherry_MX1A_1.25u_PCB
- moved TH1 7.01 mm to (273.8, 48.4)
- moved SW70 5.12 mm to (205.3, 36.4)
- moved SW71 3.86 mm to (216.7, 36.4)
- moved D1 3.81 mm to (42.7, 41.4)
- moved D10 3.81 mm to (202.7, 41.4)
- moved D11 3.81 mm to (200.2, 41.4)
- moved D12 3.81 mm to (197.6, 41.4)
- moved D13 3.81 mm to (195.1, 41.4)
- moved D14 3.81 mm to (192.6, 41.4)
- moved D15 3.81 mm to (190.0, 41.4)
- moved D16 3.81 mm to (45.2, 41.4)
- moved D17 3.81 mm to (63.0, 41.4)
- moved D18 3.81 mm to (75.7, 41.4)
- moved D19 3.81 mm to (85.9, 41.4)
- moved D2 3.81 mm to (65.6, 41.4)
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Connections:
- U1 pad 23: /COL6 -> /ROW4
- U1 pad 24: /COL7 -> /COL6
- U1 pad 25: /COL8 -> /COL7
- U1 pad 26: /COL9 -> /COL8
- U1 pad 28: Net-(R5-Pad1) -> /COL9
Routing:
- net /ROW4: track 157.7 -> 223.7 mm, vias 1 -> 0
- net Net-(R5-Pad1): track 21.5 -> 0.00 mm
- net /ROW2: track 206.6 -> 216.9 mm, vias 1 -> 0
- net /ROW3: track 203.7 -> 197.4 mm
- net /ROW0: track 219.0 -> 213.3 mm
- net Net-(LED1-Pad2): track 4.34 -> 0.00 mm
- net Net-(D4-Pad2): track 11.9 -> 16.2 mm
- net Net-(D19-Pad2): track 36.9 -> 41.1 mm
- net Net-(D18-Pad2): track 37.7 -> 41.9 mm
- net Net-(D47-Pad2): track 84.2 -> 88.3 mm
- net Net-(D45-Pad2): track 73.6 -> 77.6 mm
- net Net-(D28-Pad2): track 109.4 -> 113.3 mm
- net Net-(D29-Pad2): track 168.1 -> 171.9 mm
- net Net-(D27-Pad2): track 93.2 -> 97.0 mm
- net Net-(D34-Pad2): track 61.6 -> 65.4 mm
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Other:
- board text added: "Tartan # Through Hole Rev.1 (c)2019 Takuya Urakawa, Dm9Records"
- board text removed: "Tartan # Through Hole Rev.Alpha (c)2019 Takuya Urakawa, Dm9Records"

Commit message: rev.Alpha2
Parts:
- moved SW70 6.10 mm to (211.4, 36.4)
- moved SW71 5.08 mm to (221.8, 36.4)
- turned STAB2 to 180 degrees
- turned STAB4 to 180 degrees
- turned STAB5 to 270 degrees
- turned SW15 to 0 degrees
- turned SW56 to 0 degrees
Routing:
- net Net-(D56-Pad2): track 185.7 -> 177.5 mm
- net Net-(D15-Pad2): track 137.7 -> 132.3 mm
- net /COL2: track 273.3 -> 268.2 mm
- net /RESET: track 84.1 -> 79.4 mm
- net GND: track 9.19 -> 13.7 mm
- net /COL12: track 126.5 -> 124.0 mm
- net /COL10: track 162.2 -> 160.5 mm, vias 3 -> 2
- net /COL9: track 168.4 -> 167.0 mm
- net /COL6: track 276.0 -> 275.1 mm
- net /ROW3: track 197.4 -> 196.9 mm, vias 1 -> 0
Other:
- board text added: "Tartan # Through Hole Rev.Alpha2 (c)2019 Takuya Urakawa, Dm9Records, 5z6p.com"
- board text removed: "Tartan # Through Hole Rev.1 (c)2019 Takuya Urakawa, Dm9Records"

Commit message: update PCB rev.1
Parts:
- SW55: footprint SMKJP:SW_Cherry_MX1A_1.00u_PCB -> SMKJP:SW_Cherry_MX1A_1.75u_PCB
- SW56: footprint SMKJP:SW_Cherry_MX1A_1.75u_PCB -> SMKJP:SW_Cherry_MX1A_1.00u_PCB
- moved SW55 7.12 mm to (279.4, 118.5)
- moved SW56 7.12 mm to (305.5, 118.5)
Routing:
- net Net-(D56-Pad2): track 177.5 -> 181.0 mm
- net /COL12: track 124.0 -> 122.0 mm
Other:
- board text added: "Tartan # Through Hole Rev.1 (c)2019 Takuya Urakawa, Dm9Records, 5z6p.com"
- board text removed: "Tartan # Through Hole Rev.Alpha2 (c)2019 Takuya Urakawa, Dm9Records, 5z6p.com"
