File: pcb/tartan_bottom.kicad_pcb (KiCad board)
At the start: 2 copper layers, 285 x 117 mm, 17 parts

Commit message: rev.Alpha2
Other:
- board text added: "(c)2019 Takuya Urakawa, Dm9Records.com, 5z6p.com"
- board text removed: "(c)2019 Takuya Urakawa, Dm9Records.com"
Changed lines of the file:
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@@
     (pcbplotparams
       (layerselection 0x010f0_ffffffff)
-      (usegerberextensions false)
+      (usegerberextensions true)
       (usegerberattributes false)
       (usegerberadvancedattributes false)
@@
       (drillshape 0)
       (scaleselection 1)
-      (outputdirectory "design/"))
+      (outputdirectory "gerber/tartan_bottom"))
   )
   (net 0 "")
@@
     (effects (font (size 1 1) (thickness 0.15)) (justify left mirror))
   )
-  (gr_text "(c)2019 Takuya Urakawa, Dm9Records.com" (at 195.5 93) (layer B.SilkS)
+  (gr_text "(c)2019 Takuya Urakawa, Dm9Records.com, 5z6p.com" (at 195.5 93) (layer B.SilkS)
     (effects (font (size 1 1) (thickness 0.2)) (justify left mirror))
   )

Commit message: update PCB rev.1
Parts:
- moved G*** 2.22 mm to (172.5, 87.8)
